Commit message: 센서 tf 위치 조정

File: src/utils/erp42_visualizer/urdf/erp42.urdf.xacro (robot description, xacro)
@@ -40,8 +40,6 @@
   <xacro:disk_back_wheel prefix="right" suffix="back" roll="0" pitch="0" yall="1.5707"/>
   <xacro:disk_back_wheel prefix="left" suffix="back" roll="0" pitch="0" yall="-1.5707"/>
-  <xacro:my_camera prefix="middle" />
-  <xacro:my_camera prefix="right" />
-  <xacro:my_camera prefix="left" />
-  <xacro:my_camera prefix="back" />
+  <xacro:back_disk_wheel_joint prefix="right" suffix="back" x="-0.49" y="0.51" z="0"/>
+  <xacro:back_disk_wheel_joint prefix="left" suffix="back" x="-0.49" y="-0.51" z="0"/>
   <!-- ================== JOINTS ================== -->
   <!-- Fixed joint connecting base_link to the main structure -->
@@ -59,21 +57,16 @@
   <xacro:front_disk_wheel_joint prefix="right" suffix="front" x="0.53" y="0.51" z="0"/>
   <xacro:front_disk_wheel_joint prefix="left"  suffix="front" x="0.53" y="-0.51" z="0"/>
-  <xacro:back_disk_wheel_joint prefix="right" suffix="back" x="-0.49" y="0.51" z="0"/>
-  <xacro:back_disk_wheel_joint prefix="left" suffix="back" x="-0.49" y="-0.51" z="0"/>
-  <xacro:camera_joint prefix="middle" x="0.05" y="0" z="0.3" roll="0" pitch="0" yall="0"/>
-  <xacro:camera_joint prefix="left" x="0.05" y="0.10" z="0.3" roll="0" pitch="0" yall="0.785"/>
-  <xacro:camera_joint prefix="right" x="0.05" y="-0.10" z="0.3" roll="0" pitch="0" yall="-0.785"/>
-  <xacro:camera_joint prefix="back" x="-0.05" y="0" z="0.4" roll="0" pitch="0" yall="3.1414"/>
   <!-- =================================================================== -->
   <!--                      CUSTOM SENSORS                                 -->
   <!-- =================================================================== -->
-  <!-- 1. IMU SENSOR (BLUE BOX) -->
+  <!-- 1. IMU SENSOR -->
   <link name="imu_link">
     <visual>
+      <!-- Shape: <box>, <cylinder>, or <sphere> -->
       <geometry>
         <box size="0.05 0.05 0.02"/>
       </geometry>
-      <material name="blue">
-        <color rgba="0.0 0.0 1.0 1.0"/>
+      <material name="red">
+        <color rgba="1.0 0.0 0.0 1.0"/>
       </material>
     </visual>
@@ -82,12 +75,12 @@
     <parent link="base_link"/>
     <child link="imu_link"/>
-    <!-- Position and orientation relative to base_link. Modify as needed. -->
-    <origin xyz="0.3 0 0.4" rpy="0 0 0"/>
+    <!-- Position (xyz) and Orientation (rpy) -->
+    <origin xyz="0.0 0.0 1.12" rpy="0 0 0"/>
   </joint>
-  <!-- 2. GPS SENSOR (GREEN BOX) -->
+  <!-- 2. GPS SENSOR -->
   <link name="gps_link">
     <visual>
       <geometry>
-        <box size="0.1 0.1 0.05"/>
+        <box size="0.05 0.05 0.02"/>
       </geometry>
       <material name="green">
@@ -99,14 +92,15 @@
     <parent link="base_link"/>
     <child link="gps_link"/>
-    <origin xyz="-0.5 0 0.8" rpy="0 0 0"/>
+    <!-- Positioned on the rear of the roof -->
+    <origin xyz="0.2 0.0 1.27" rpy="0 0 0"/>
   </joint>
-  <!-- 3. LIDAR SENSOR (RED CYLINDER) -->
+  <!-- 3. LIDAR SENSOR -->
   <link name="lidar_link">
     <visual>
       <geometry>
-        <cylinder radius="0.05" length="0.08"/>
+        <cylinder radius="0.06" length="0.08"/>
       </geometry>
-      <material name="red">
-        <color rgba="1.0 0.0 0.0 1.0"/>
+      <material name="blue">
+        <color rgba="0.0 0.0 1.0 1.0"/>
       </material>
     </visual>
@@ -115,5 +109,6 @@
     <parent link="base_link"/>
     <child link="lidar_link"/>
-    <origin xyz="0.0 0 0.9" rpy="0 0 0"/>
+    <!-- Positioned on the center of the roof -->
+    <origin xyz="1.3 0.0 0.42" rpy="0 0 0"/>
   </joint>
 </robot>

Commit message: patchworkpp+adaptive clustering

File: src/utils/erp42_visualizer/urdf/erp42.urdf.xacro (robot description, xacro)
@@ -96,5 +96,5 @@
   </joint>
   <!-- 3. LIDAR SENSOR -->
-  <link name="lidar_link">
+  <link name="velodyne">
     <visual>
       <geometry>
@@ -108,5 +108,5 @@
   <joint name="lidar_joint" type="fixed">
     <parent link="base_link"/>
-    <child link="lidar_link"/>
+    <child link="velodyne"/>
     <!-- Positioned on the center of the roof -->
     <origin xyz="1.3 0.0 0.42" rpy="0 0 0"/>

Commit message: 본선 맵 배달 구간 변경

File: src/utils/erp42_visualizer/urdf/erp42.urdf.xacro (robot description, xacro)
@@ -47,6 +47,6 @@
       <parent link="base_link"/>
       <child link="structure"/>
-      <!-- Move structure forward by 0.49m to place base_link at the rear axle center -->
-      <origin xyz="0.49 0 0" rpy="0 0 0"/>
+      <!-- Move structure forward by 0.49m and raise by wheel radius to sit above ground -->
+      <origin xyz="0.49 0 ${wheel_radius}" rpy="0 0 0"/>
   </joint>
   <!-- Macro-generated joints (Wheel actuation and steering) -->
@@ -112,3 +112,28 @@
     <origin xyz="1.3 0.0 0.42" rpy="0 0 0"/>
   </joint>
+  <!-- 4. CAMERA SENSOR (adds TF for 'camera' to match CameraInfo frame_id) -->
+  <link name="camera">
+    <visual>
+      <geometry>
+        <box size="0.04 0.04 0.04"/>
+      </geometry>
+      <material name="grey">
+        <color rgba="0.5 0.5 0.5 1.0"/>
+      </material>
+    </visual>
+  </link>
+  <joint name="camera_joint" type="fixed">
+    <parent link="base_link"/>
+    <child link="camera"/>
+    <!-- Approximate front-mounted camera pose (adjust as needed) -->
+    <origin xyz="0.70 0.00 1.20" rpy="0 0 0"/>
+  </joint>
+  <!-- Optional optical frame for visualization conventions -->
+  <link name="camera_optical_frame"/>
+  <joint name="camera_optical_joint" type="fixed">
+    <parent link="camera"/>
+    <child link="camera_optical_frame"/>
+    <!-- REP-103: optical frame has Z forward, X right, Y down -->
+    <origin xyz="0 0 0" rpy="-1.57079632679 0 -1.57079632679"/>
+  </joint>
 </robot>

File: src/utils/erp42_visualizer/urdf/macros_erp42.xacro (robot description, xacro)
@@ -34,6 +34,5 @@
  <!-- Wheel joint macros -->
   <xacro:macro name="wheel_front_joint" params="prefix suffix x y z ">
-   <joint name="${prefix}_${suffix}_wheel_joint" type="continuous">
-      <axis xyz="0 1 0" />
+   <joint name="${prefix}_${suffix}_wheel_joint" type="fixed">
       <parent link="${prefix}_${suffix}_disk_wheel"/>
       <child link="${prefix}_${suffix}_wheel"/>
@@ -42,6 +41,5 @@
   </xacro:macro>
   <xacro:macro name="wheel_back_joint" params="prefix suffix x y z ">
-   <joint name="${prefix}_${suffix}_wheel_joint" type="continuous">
-      <axis xyz="0 1 0" />
+   <joint name="${prefix}_${suffix}_wheel_joint" type="fixed">
       <parent link="${prefix}_${suffix}_disk_wheel"/>
       <child link="${prefix}_${suffix}_wheel"/>
@@ -94,10 +92,8 @@
 <!-- Disk joint macros -->
  <xacro:macro name="front_disk_wheel_joint" params=" prefix suffix x y z">
-  <joint name="${prefix}_${suffix}_disk_wheel_joint" type="revolute">
-      <axis xyz="0 0 1" />
+  <joint name="${prefix}_${suffix}_disk_wheel_joint" type="fixed">
       <parent link="structure"/>
       <child link="${prefix}_${suffix}_disk_wheel"/>
       <origin xyz="${x} ${y} ${z}" />
-      <limit effort="1000.0" lower="-0.4" upper="0.4" velocity="0.5"/>
   </joint>
  </xacro:macro>

Commit message: global planner, 시각화 수정

File: src/utils/erp42_visualizer/urdf/erp42.urdf.xacro (robot description, xacro)
@@ -110,5 +110,5 @@
     <child link="velodyne"/>
     <!-- Positioned on the center of the roof -->
-    <origin xyz="1.3 0.0 0.42" rpy="0 0 0"/>
+    <origin xyz="1.3 0.0 0.7" rpy="0 0 0"/>
   </joint>
   <!-- 4. CAMERA SENSOR (adds TF for 'camera' to match CameraInfo frame_id) -->

Commit message: global planner world-> map, /autocar/goals 모두 통합 후 다시 보간

File: src/utils/erp42_visualizer/urdf/erp42.urdf.xacro (robot description, xacro)
@@ -65,8 +65,8 @@
       <!-- Shape: <box>, <cylinder>, or <sphere> -->
       <geometry>
-        <box size="0.05 0.05 0.02"/>
+        <box size="0.05 0.05 0.03"/>
       </geometry>
       <material name="red">
-        <color rgba="1.0 0.0 0.0 1.0"/>
+        <color rgba="1.0 0.0 0.0 0.9"/>
       </material>
     </visual>
@@ -76,5 +76,5 @@
     <child link="imu_link"/>
     <!-- Position (xyz) and Orientation (rpy) -->
-    <origin xyz="0.0 0.0 1.12" rpy="0 0 0"/>
+    <origin xyz="0.05 0.0 1.40" rpy="0 0 0"/>
   </joint>
   <!-- 2. GPS SENSOR -->
@@ -82,8 +82,8 @@
     <visual>
       <geometry>
-        <box size="0.05 0.05 0.02"/>
+        <box size="0.12 0.06 0.03"/>
       </geometry>
       <material name="green">
-        <color rgba="0.0 1.0 0.0 1.0"/>
+        <color rgba="0.0 1.0 0.0 0.9"/>
       </material>
     </visual>
@@ -93,5 +93,5 @@
     <child link="gps_link"/>
     <!-- Positioned on the rear of the roof -->
-    <origin xyz="0.2 0.0 1.27" rpy="0 0 0"/>
+    <origin xyz="0.40 0.0 1.40" rpy="0 0 0"/>
   </joint>
   <!-- 3. LIDAR SENSOR -->
@@ -99,8 +99,8 @@
     <visual>
       <geometry>
-        <cylinder radius="0.06" length="0.08"/>
+        <cylinder radius="0.1" length="0.1"/>
       </geometry>
       <material name="blue">
-        <color rgba="0.0 0.0 1.0 1.0"/>
+        <color rgba="0.0 0.0 1.0 0.9"/>
       </material>
     </visual>
@@ -110,28 +110,28 @@
     <child link="velodyne"/>
     <!-- Positioned on the center of the roof -->
-    <origin xyz="1.3 0.0 0.7" rpy="0 0 0"/>
+    <origin xyz="1.33 0.0 0.7" rpy="0 0 0"/>
   </joint>
   <!-- 4. CAMERA SENSOR (adds TF for 'camera' to match CameraInfo frame_id) -->
-  <link name="camera">
+  <link name="camera_front_link">
     <visual>
       <geometry>
-        <box size="0.04 0.04 0.04"/>
+        <box size="0.03 0.10 0.03"/>
       </geometry>
       <material name="grey">
-        <color rgba="0.5 0.5 0.5 1.0"/>
+        <color rgba="0.5 0.5 0.5 0.9"/>
       </material>
     </visual>
   </link>
-  <joint name="camera_joint" type="fixed">
+  <joint name="camera_front_joint" type="fixed">
     <parent link="base_link"/>
-    <child link="camera"/>
+    <child link="camera_front_link"/>
     <!-- Approximate front-mounted camera pose (adjust as needed) -->
-    <origin xyz="0.70 0.00 1.20" rpy="0 0 0"/>
+    <origin xyz="0.58 0.00 1.33" rpy="0 0 0"/>
   </joint>
   <!-- Optional optical frame for visualization conventions -->
-  <link name="camera_optical_frame"/>
-  <joint name="camera_optical_joint" type="fixed">
-    <parent link="camera"/>
-    <child link="camera_optical_frame"/>
+  <link name="camera_front_optical_frame"/>
+  <joint name="camera_front_optical_joint" type="fixed">
+    <parent link="camera_front_link"/>
+    <child link="camera_front_optical_frame"/>
     <!-- REP-103: optical frame has Z forward, X right, Y down -->
     <origin xyz="0 0 0" rpy="-1.57079632679 0 -1.57079632679"/>
